File: hardware/playboard/3ch_fetdriver.sch (KiCad schematic (older format))
At the start: 6 parts

Commit message: Worked some more on the playboard
Parts:
- gave numbers to parts that had none: 6
Changed lines of the file:
@@
-EESchema Schematic File Version 2  date Sat 08 Jun 2013 01:37:28 AM CEST
+EESchema Schematic File Version 2
 LIBS:power
 LIBS:device
@@
 LIBS:usb_micro-b
 LIBS:microphone
+LIBS:crf
 LIBS:playboard1-cache
 EELAYER 27 0
@@
 Sheet 2 7
 Title ""
-Date "7 jun 2013"
+Date "16 jun 2013"
 Rev ""
 Comp ""
@@
 $EndDescr
 $Comp
-L MOSFET_N Q?
+L MOSFET_N Q3
 U 1 1 51B25338
 P 2900 1850
-F 0 "Q?" H 2910 2020 60  0000 R CNN
+AR Path="/51B25330/51B25338" Ref="Q3"  Part="1"
+AR Path="/51B279F6/51B25338" Ref="Q6"  Part="1"
+AR Path="/51B287A5/51B25338" Ref="Q9"  Part="1"
+F 0 "Q6" H 2910 2020 60  0000 R CNN
 F 1 "MOSFET_N" H 2910 1700 60  0000 R CNN
 F 2 "~" H 2900 1850 60  0000 C CNN
@@
 $EndComp
 $Comp
-L R R?
+L R R19
 U 1 1 51B25347
 P 2350 2250
-F 0 "R?" V 2430 2250 40  0000 C CNN
+AR Path="/51B25330/51B25347" Ref="R19"  Part="1"
+AR Path="/51B279F6/51B25347" Ref="R22"  Part="1"
+AR Path="/51B287A5/51B25347" Ref="R25"  Part="1"
+F 0 "R22" V 2430 2250 40  0000 C CNN
 F 1 "R" V 2357 2251 40  0000 C CNN
 F 2 "~" V 2280 2250 30  0000 C CNN
@@
 	3000 2050 3000 2600
 $Comp
-L MOSFET_N Q?
+L MOSFET_N Q4
 U 1 1 51B2558E
 P 4250 1850
-F 0 "Q?" H 4260 2020 60  0000 R CNN
+AR Path="/51B25330/51B2558E" Ref="Q4"  Part="1"
+AR Path="/51B279F6/51B2558E" Ref="Q7"  Part="1"
+AR Path="/51B287A5/51B2558E" Ref="Q10"  Part="1"
+F 0 "Q7" H 4260 2020 60  0000 R CNN
 F 1 "MOSFET_N" H 4260 1700 60  0000 R CNN
 F 2 "~" H 4250 1850 60  0000 C CNN
@@
 $EndComp
 $Comp
-L R R?
+L R R20
 U 1 1 51B25594
 P 3700 2250
-F 0 "R?" V 3780 2250 40  0000 C CNN
+AR Path="/51B25330/51B25594" Ref="R20"  Part="1"
+AR Path="/51B279F6/51B25594" Ref="R23"  Part="1"
+AR Path="/51B287A5/51B25594" Ref="R26"  Part="1"
+F 0 "R23" V 3780 2250 40  0000 C CNN
 F 1 "R" V 3707 2251 40  0000 C CNN
 F 2 "~" V 3630 2250 30  0000 C CNN
@@
 	4350 2050 4350 2600
 $Comp
-L MOSFET_N Q?
+L MOSFET_N Q5
 U 1 1 51B255A6
 P 5650 1850
-F 0 "Q?" H 5660 2020 60  0000 R CNN
+AR Path="/51B25330/51B255A6" Ref="Q5"  Part="1"
+AR Path="/51B279F6/51B255A6" Ref="Q8"  Part="1"
+AR Path="/51B287A5/51B255A6" Ref="Q11"  Part="1"
+F 0 "Q8" H 5660 2020 60  0000 R CNN
 F 1 "MOSFET_N" H 5660 1700 60  0000 R CNN
 F 2 "~" H 5650 1850 60  0000 C CNN
@@
 $EndComp
 $Comp
-L R R?
+L R R21
 U 1 1 51B255AC
 P 5100 2250
-F 0 "R?" V 5180 2250 40  0000 C CNN
+AR Path="/51B25330/51B255AC" Ref="R21"  Part="1"
+AR Path="/51B279F6/51B255AC" Ref="R24"  Part="1"
+AR Path="/51B287A5/51B255AC" Ref="R27"  Part="1"
+F 0 "R24" V 5180 2250 40  0000 C CNN
 F 1 "R" V 5107 2251 40  0000 C CNN
 F 2 "~" V 5030 2250 30  0000 C CNN

Commit message: Comitting before rerouting
Changed lines of the file:
@@
 AR Path="/51B279F6/51B25338" Ref="Q6"  Part="1"
 AR Path="/51B287A5/51B25338" Ref="Q9"  Part="1"
-F 0 "Q6" H 2910 2020 60  0000 R CNN
+F 0 "Q9" H 2910 2020 60  0000 R CNN
 F 1 "MOSFET_N" H 2910 1700 60  0000 R CNN
 F 2 "~" H 2900 1850 60  0000 C CNN
@@
 AR Path="/51B279F6/51B25347" Ref="R22"  Part="1"
 AR Path="/51B287A5/51B25347" Ref="R25"  Part="1"
-F 0 "R22" V 2430 2250 40  0000 C CNN
+F 0 "R25" V 2430 2250 40  0000 C CNN
 F 1 "R" V 2357 2251 40  0000 C CNN
 F 2 "~" V 2280 2250 30  0000 C CNN
@@
 AR Path="/51B279F6/51B2558E" Ref="Q7"  Part="1"
 AR Path="/51B287A5/51B2558E" Ref="Q10"  Part="1"
-F 0 "Q7" H 4260 2020 60  0000 R CNN
+F 0 "Q10" H 4260 2020 60  0000 R CNN
 F 1 "MOSFET_N" H 4260 1700 60  0000 R CNN
 F 2 "~" H 4250 1850 60  0000 C CNN
@@
 AR Path="/51B279F6/51B25594" Ref="R23"  Part="1"
 AR Path="/51B287A5/51B25594" Ref="R26"  Part="1"
-F 0 "R23" V 3780 2250 40  0000 C CNN
+F 0 "R26" V 3780 2250 40  0000 C CNN
 F 1 "R" V 3707 2251 40  0000 C CNN
 F 2 "~" V 3630 2250 30  0000 C CNN
@@
 AR Path="/51B279F6/51B255A6" Ref="Q8"  Part="1"
 AR Path="/51B287A5/51B255A6" Ref="Q11"  Part="1"
-F 0 "Q8" H 5660 2020 60  0000 R CNN
+F 0 "Q11" H 5660 2020 60  0000 R CNN
 F 1 "MOSFET_N" H 5660 1700 60  0000 R CNN
 F 2 "~" H 5650 1850 60  0000 C CNN
@@
 AR Path="/51B279F6/51B255AC" Ref="R24"  Part="1"
 AR Path="/51B287A5/51B255AC" Ref="R27"  Part="1"
-F 0 "R24" V 5180 2250 40  0000 C CNN
+F 0 "R27" V 5180 2250 40  0000 C CNN
 F 1 "R" V 5107 2251 40  0000 C CNN
 F 2 "~" V 5030 2250 30  0000 C CNN
