File: hardware/playboard/playboard1.sch (KiCad schematic (older format))
At the start: 43 parts

Commit message: Worked some more on the playboard
Parts:
- removed C?: CP, ~, symbol CP
- added C10: 10 nF, ~, symbol C
- added C14, C9: 10 µF, ~, symbol C
- added C15: 100 nF, ~, symbol C
- added C8: 2.2 µF, ~, symbol C
- added D7: Pink, ~, symbol LED
- added H1: DRV8833, ~, symbol DRV8833
- added JP1, JP2: JUMPER3, ~, symbol JUMPER3
- added P1, P5: CONN_6, ~, symbol CONN_6
- added P10, P4: CONN_4, ~, symbol CONN_4
- added P2, P3: CONN_2, ~, symbol CONN_2
- added Q1: NPN, ~, symbol NPN
- added R1, R10: 10 kΩ, ~, symbol R
- added R18: 120 Ω, ~, symbol R
- added R37, R38: 100 kΩ, ~, symbol R
- added R8: 4.7 kΩ, ~, symbol R
- C1, C11, C2, C3, C4, C5, C6, C7: renamed from C?; value C -> 100 nF
- C12: renamed from C?; value CP -> 100 µF
- C13: renamed from C?; value CP -> 22 µF
- D1, D6: renamed from D?; value LED -> Red
- D2: renamed from D?; value LED -> Green
- D5: renamed from D?; value LED -> Orange
- R11, R13, R2, R3, R4, R6, R7, R9: renamed from R?; value R -> 10 kΩ
- R12: renamed from R?; value R -> 100 kΩ
- R14, R15, R16: renamed from R?; value R -> 290 Ω
- R17: renamed from R?; value R -> 1 kΩ
- R5: renamed from R?; value R -> 4.7 kΩ
- gave numbers to parts that had none: 14
Connections:
- net labels added: BO1, BO2, BO3, Board_NRST, DRV_VINT, DRV_nFault, DRV_nSLEEP, Debug_LED, GO1, GO2, GO3, I2C_EXTPULL, I2C_PULL, PO_H, PO_L, RO1, RO2, RO3, RX2, TX2
- wire segments 97 -> 218
- no-connect marks 6 -> 22
Other:
- note added: "GPIO"
- moved on the sheet: C1, C11, C12, C2, C3, C4, C5, C6, D1, D2, D3, D4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

Commit message: Comitting before rerouting
Parts:
- added J1: SMA, SMA, symbol SMA
- added R?: 0 Ω, ~, symbol R
- added U7: RF2400-NANO, ~, symbol RF2400-NANO
Connections:
- net labels added: R_CE, R_IRQ, R_MISO, R_MOSI, R_NSS, R_SCK
- wire segments 218 -> 173
- no-connect marks 22 -> 16

Commit message: Redesigned board for playboard.
Parts:
- removed R?: 0 Ω, ~, symbol R
Connections:
- wire segments 173 -> 172
Changed lines of the file:
@@
 USBD+
 $Comp
-L GND #PWR1
+L GND #PWR01
 U 1 1 51B22BC9
 P 1400 2650
-F 0 "#PWR1" H 1400 2650 30  0001 C CNN
+F 0 "#PWR01" H 1400 2650 30  0001 C CNN
 F 1 "GND" H 1400 2580 30  0001 C CNN
 F 2 "" H 1400 2650 60  0000 C CNN
@@
 $EndComp
 $Comp
-L GND #PWR21
+L GND #PWR02
 U 1 1 51B22BF4
 P 13250 8800
-F 0 "#PWR21" H 13250 8800 30  0001 C CNN
+F 0 "#PWR02" H 13250 8800 30  0001 C CNN
 F 1 "GND" H 13250 8730 30  0001 C CNN
 F 2 "" H 13250 8800 60  0000 C CNN
@@
 NRST
 $Comp
-L GND #PWR5
+L GND #PWR03
 U 1 1 51B22D53
 P 4150 2100
-F 0 "#PWR5" H 4150 2100 30  0001 C CNN
+F 0 "#PWR03" H 4150 2100 30  0001 C CNN
 F 1 "GND" H 4150 2030 30  0001 C CNN
 F 2 "" H 4150 2100 60  0000 C CNN
@@
 USB Powered LED's
 $Comp
-L GND #PWR10
+L GND #PWR04
 U 1 1 51B22E3E
 P 8100 4350
-F 0 "#PWR10" H 8100 4350 30  0001 C CNN
+F 0 "#PWR04" H 8100 4350 30  0001 C CNN
 F 1 "GND" H 8100 4280 30  0001 C CNN
 F 2 "" H 8100 4350 60  0000 C CNN
@@
 $EndComp
 $Comp
-L GND #PWR12
+L GND #PWR05
 U 1 1 51B238E4
 P 8950 2250
-F 0 "#PWR12" H 8950 2250 30  0001 C CNN
+F 0 "#PWR05" H 8950 2250 30  0001 C CNN
 F 1 "GND" H 8950 2180 30  0001 C CNN
 F 2 "" H 8950 2250 60  0000 C CNN
@@
 VCC_3V3
 $Comp
-L GND #PWR4
+L GND #PWR06
 U 1 1 51B23E99
 P 4100 6300
-F 0 "#PWR4" H 4100 6300 30  0001 C CNN
+F 0 "#PWR06" H 4100 6300 30  0001 C CNN
 F 1 "GND" H 4100 6230 30  0001 C CNN
 F 2 "" H 4100 6300 60  0000 C CNN
@@
 VCC_3V3
 $Comp
-L GND #PWR6
+L GND #PWR07
 U 1 1 51B2407C
 P 4700 7350
-F 0 "#PWR6" H 4700 7350 30  0001 C CNN
+F 0 "#PWR07" H 4700 7350 30  0001 C CNN
 F 1 "GND" H 4700 7280 30  0001 C CNN
 F 2 "" H 4700 7350 60  0000 C CNN
@@
 $EndComp
 $Comp
-L GND #PWR2
+L GND #PWR08
 U 1 1 51B245D7
 P 1550 7600
-F 0 "#PWR2" H 1550 7600 30  0001 C CNN
+F 0 "#PWR08" H 1550 7600 30  0001 C CNN
 F 1 "GND" H 1550 7530 30  0001 C CNN
 F 2 "" H 1550 7600 60  0000 C CNN
@@
 $EndComp
 $Comp
-L GND #PWR13
+L GND #PWR09
 U 1 1 51B24AF2
 P 9350 4400
-F 0 "#PWR13" H 9350 4400 30  0001 C CNN
+F 0 "#PWR09" H 9350 4400 30  0001 C CNN
 F 1 "GND" H 9350 4330 30  0001 C CNN
 F 2 "" H 9350 4400 60  0000 C CNN
@@
 $EndSheet
 $Comp
-L GND #PWR20
+L GND #PWR010
 U 1 1 51B28A28
 P 12150 7000
-F 0 "#PWR20" H 12150 7000 30  0001 C CNN
+F 0 "#PWR010" H 12150 7000 30  0001 C CNN
 F 1 "GND" H 12150 6930 30  0001 C CNN
 F 2 "" H 12150 7000 60  0000 C CNN
@@
 $EndComp
 $Comp
-L GND #PWR8
+L GND #PWR011
 U 1 1 51B27ED0
 P 6950 2150
-F 0 "#PWR8" H 6950 2150 30  0001 C CNN
+F 0 "#PWR011" H 6950 2150 30  0001 C CNN
 F 1 "GND" H 6950 2080 30  0001 C CNN
 F 2 "" H 6950 2150 60  0000 C CNN
@@
 $EndComp
 $Comp
-L GND #PWR3
+L GND #PWR012
 U 1 1 51BCF415
 P 2350 9700
-F 0 "#PWR3" H 2350 9700 30  0001 C CNN
+F 0 "#PWR012" H 2350 9700 30  0001 C CNN
 F 1 "GND" H 2350 9630 30  0001 C CNN
 F 2 "" H 2350 9700 60  0000 C CNN
@@
 $EndComp
 $Comp
-L GND #PWR9
+L GND #PWR013
 U 1 1 51BD2AE0
 P 7600 7450
-F 0 "#PWR9" H 7600 7450 30  0001 C CNN
+F 0 "#PWR013" H 7600 7450 30  0001 C CNN
 F 1 "GND" H 7600 7380 30  0001 C CNN
 F 2 "" H 7600 7450 60  0000 C CNN
@@
 DRV_nFault
 $Comp
-L GND #PWR16
+L GND #PWR014
 U 1 1 51BD6366
 P 10300 6500
-F 0 "#PWR16" H 10300 6500 30  0001 C CNN
+F 0 "#PWR014" H 10300 6500 30  0001 C CNN
 F 1 "GND" H 10300 6430 30  0001 C CNN
 F 2 "" H 10300 6500 60  0000 C CNN
@@
 $EndComp
 $Comp
-L GND #PWR7
+L GND #PWR015
 U 1 1 51BD71F6
 P 5450 9300
-F 0 "#PWR7" H 5450 9300 30  0001 C CNN
+F 0 "#PWR015" H 5450 9300 30  0001 C CNN
 F 1 "GND" H 5450 9230 30  0001 C CNN
 F 2 "" H 5450 9300 60  0000 C CNN
@@
 $EndComp
 $Comp
-L GND #PWR22
+L GND #PWR016
 U 1 1 51BDA520
 P 14700 8650
-F 0 "#PWR22" H 14700 8650 30  0001 C CNN
+F 0 "#PWR016" H 14700 8650 30  0001 C CNN
 F 1 "GND" H 14700 8580 30  0001 C CNN
 F 2 "" H 14700 8650 60  0000 C CNN
@@
 $EndComp
 $Comp
-L GND #PWR17
+L GND #PWR017
 U 1 1 51BE03EB
 P 10700 9550
-F 0 "#PWR17" H 10700 9550 30  0001 C CNN
+F 0 "#PWR017" H 10700 9550 30  0001 C CNN
 F 1 "GND" H 10700 9480 30  0001 C CNN
 F 2 "" H 10700 9550 60  0000 C CNN
@@
 VCC_3V3
 $Comp
-L GND #PWR19
+L GND #PWR018
 U 1 1 51BE10C1
 P 11050 8800
-F 0 "#PWR19" H 11050 8800 30  0001 C CNN
+F 0 "#PWR018" H 11050 8800 30  0001 C CNN
 F 1 "GND" H 11050 8730 30  0001 C CNN
 F 2 "" H 11050 8800 60  0000 C CNN
@@
 VCC_3V3
 $Comp
-L GND #PWR18
+L GND #PWR019
 U 1 1 51BE671B
 P 10700 10300
-F 0 "#PWR18" H 10700 10300 30  0001 C CNN
+F 0 "#PWR019" H 10700 10300 30  0001 C CNN
 F 1 "GND" H 10700 10230 30  0001 C CNN
 F 2 "" H 10700 10300 60  0000 C CNN
@@
 R_IRQ
 $Comp
-L GND #PWR11
+L GND #PWR020
 U 1 1 51BE0DE3
 P 8200 9000
-F 0 "#PWR11" H 8200 9000 30  0001 C CNN
+F 0 "#PWR020" H 8200 9000 30  0001 C CNN
 F 1 "GND" H 8200 8930 30  0001 C CNN
 F 2 "" H 8200 9000 60  0000 C CNN
@@
 	8200 8850 8200 9000
 $Comp
-L GND #PWR14
+L GND #PWR021
 U 1 1 51BE1317
 P 9350 8500
-F 0 "#PWR14" H 9350 8500 30  0001 C CNN
+F 0 "#PWR021" H 9350 8500 30  0001 C CNN
 F 1 "GND" H 9350 8430 30  0001 C CNN
 F 2 "" H 9350 8500 60  0000 C CNN
@@
 $EndComp
 $Comp
-L GND #PWR15
+L GND #PWR022
 U 1 1 51BE1CC0
 P 9750 8500
-F 0 "#PWR15" H 9750 8500 30  0001 C CNN
+F 0 "#PWR022" H 9750 8500 30  0001 C CNN
 F 1 "GND" H 9750 8430 30  0001 C CNN
 F 2 "" H 9750 8500 60  0000 C CNN
@@
 	9750 7650 9800 7650
 Connection ~ 9800 7700
-$Comp
-L R R?
-U 1 1 51BE30FD
-P 9550 8150
-F 0 "R?" V 9630 8150 40  0000 C CNN
-F 1 "0 Ω" V 9557 8151 40  0000 C CNN
-F 2 "~" V 9480 8150 30  0000 C CNN
-F 3 "~" H 9550 8150 30  0000 C CNN
-	1    9550 8150
-	1    0    0    -1
-$EndComp
-Wire Wire Line
-	9550 7900 9550 7850
-Wire Wire Line
-	9550 8450 9550 8400
+Wire Wire Line
+	9550 7850 9550 8450
 $EndSCHEMATC
