File: hardware/playboard/rgbled.sch (KiCad schematic (older format))
At the start: 4 parts

Commit message: Added some new hardware, included some code objects forgotten locally.
Parts:
- gave numbers to parts that had none: 4
Changed lines of the file:
@@
-EESchema Schematic File Version 2  date Sat 08 Jun 2013 01:37:28 AM CEST
+EESchema Schematic File Version 2  date Fri 14 Jun 2013 08:33:45 PM CEST
 LIBS:power
 LIBS:device
@@
 Sheet 5 7
 Title ""
-Date "7 jun 2013"
+Date "14 jun 2013"
 Rev ""
 Comp ""
@@
 $EndDescr
 $Comp
-L PLCC6XRGBCT U?
+L PLCC6XRGBCT U4
 U 1 1 51B29101
 P 4350 3200
-F 0 "U?" H 4350 3650 60  0000 C CNN
+AR Path="/51B29079/51B29101" Ref="U4"  Part="1"
+AR Path="/51B29C83/51B29101" Ref="U5"  Part="1"
+AR Path="/51B2A046/51B29101" Ref="U6"  Part="1"
+F 0 "U4" H 4350 3650 60  0000 C CNN
 F 1 "PLCC6XRGBCT" H 4350 2700 60  0000 C CNN
 F 2 "" H 4350 3200 60  0000 C CNN
@@
 $EndComp
 $Comp
-L R R?
+L R R24
 U 1 1 51B29110
 P 3750 2900
-F 0 "R?" V 3830 2900 40  0000 C CNN
+AR Path="/51B29079/51B29110" Ref="R24"  Part="1"
+AR Path="/51B29C83/51B29110" Ref="R27"  Part="1"
+AR Path="/51B2A046/51B29110" Ref="R30"  Part="1"
+F 0 "R24" V 3830 2900 40  0000 C CNN
 F 1 "R" V 3757 2901 40  0000 C CNN
 F 2 "~" V 3680 2900 30  0000 C CNN
@@
 $EndComp
 $Comp
-L R R?
+L R R25
 U 1 1 51B29140
 P 3750 3150
-F 0 "R?" V 3830 3150 40  0000 C CNN
+AR Path="/51B29079/51B29140" Ref="R25"  Part="1"
+AR Path="/51B29C83/51B29140" Ref="R28"  Part="1"
+AR Path="/51B2A046/51B29140" Ref="R31"  Part="1"
+F 0 "R25" V 3830 3150 40  0000 C CNN
 F 1 "R" V 3757 3151 40  0000 C CNN
 F 2 "~" V 3680 3150 30  0000 C CNN
@@
 $EndComp
 $Comp
-L R R?
+L R R26
 U 1 1 51B29146
 P 3750 3400
-F 0 "R?" V 3830 3400 40  0000 C CNN
+AR Path="/51B29079/51B29146" Ref="R26"  Part="1"
+AR Path="/51B29C83/51B29146" Ref="R29"  Part="1"
+AR Path="/51B2A046/51B29146" Ref="R32"  Part="1"
+F 0 "R26" V 3830 3400 40  0000 C CNN
 F 1 "R" V 3757 3401 40  0000 C CNN
 F 2 "~" V 3680 3400 30  0000 C CNN
