File: hardware/5strip/3ch_fetdriver.sch (KiCad schematic (older format))
At the start: 6 parts, among them Q2 MOS_N_GDS, Q3 MOS_N_GDS, Q4 MOS_N_GDS

Commit message: Updated timer registers in rxlamp code
Changed lines of the file:
@@
-EESchema Schematic File Version 2  date Sat 29 Jun 2013 10:13:31 AM CEST
+EESchema Schematic File Version 2  date Tue 02 Jul 2013 07:50:22 AM CEST
 LIBS:power
 LIBS:device
@@
 Sheet 4 6
 Title ""
-Date "29 jun 2013"
+Date "2 jul 2013"
 Rev ""
 Comp ""
@@
 AR Path="/51CCC7CF/51B25347" Ref="R22"  Part="1"
 AR Path="/51CCCDF1/51B25347" Ref="R25"  Part="1"
-F 0 "R19" V 2430 2250 40  0000 C CNN
+F 0 "R25" V 2430 2250 40  0000 C CNN
 F 1 "R" V 2357 2251 40  0000 C CNN
 F 2 "~" V 2280 2250 30  0000 C CNN
@@
 AR Path="/51CCC7CF/51B25594" Ref="R23"  Part="1"
 AR Path="/51CCCDF1/51B25594" Ref="R26"  Part="1"
-F 0 "R20" V 3780 2250 40  0000 C CNN
+F 0 "R26" V 3780 2250 40  0000 C CNN
 F 1 "R" V 3707 2251 40  0000 C CNN
 F 2 "~" V 3630 2250 30  0000 C CNN
@@
 AR Path="/51CCC7CF/51B255AC" Ref="R24"  Part="1"
 AR Path="/51CCCDF1/51B255AC" Ref="R27"  Part="1"
-F 0 "R21" V 5180 2250 40  0000 C CNN
+F 0 "R27" V 5180 2250 40  0000 C CNN
 F 1 "R" V 5107 2251 40  0000 C CNN
 F 2 "~" V 5030 2250 30  0000 C CNN
@@
 AR Path="/51CCC7CF/51CEB3AA" Ref="Q11"  Part="1"
 AR Path="/51CCCDF1/51CEB3AA" Ref="Q14"  Part="1"
-F 0 "Q8" H 2910 2020 60  0000 R CNN
+F 0 "Q14" H 2910 2020 60  0000 R CNN
 F 1 "MOS_N_GDS" H 2910 1700 60  0000 R CNN
 F 2 "~" H 2900 1850 60  0000 C CNN
@@
 AR Path="/51CCC7CF/51CEB3B7" Ref="Q12"  Part="1"
 AR Path="/51CCCDF1/51CEB3B7" Ref="Q15"  Part="1"
-F 0 "Q9" H 4260 2020 60  0000 R CNN
+F 0 "Q15" H 4260 2020 60  0000 R CNN
 F 1 "MOS_N_GDS" H 4260 1700 60  0000 R CNN
 F 2 "~" H 4250 1850 60  0000 C CNN
@@
 AR Path="/51CCC7CF/51CEB3BD" Ref="Q13"  Part="1"
 AR Path="/51CCCDF1/51CEB3BD" Ref="Q16"  Part="1"
-F 0 "Q10" H 5660 2020 60  0000 R CNN
+F 0 "Q16" H 5660 2020 60  0000 R CNN
 F 1 "MOS_N_GDS" H 5660 1700 60  0000 R CNN
 F 2 "~" H 5650 1850 60  0000 C CNN
